File: pcb/clock.sch (EAGLE design)
At the start: 72 parts, among them IC1 STM32F072C8T6, IC2 REG1117, IC3 24C64ST, U1 DS18B20, X3 USB-MICROB

Commit message: added bom
Parts:
- removed C10, C4, C5, C9: (no value), clock:C-USC1210
- C1, C6, C7, C8: value (none) -> 100nF
- C11, C12: value (none) -> 20p
- C13, C14, C2: value (none) -> 47uF
- C17, C3: value (none) -> 20pF
- L1: value (none) -> 33nH
- R1, R13, R16, R17, R2, R3, R7, R8, R9: value (none) -> 4K7
- R11, R12, R4: value (none) -> 10
- R14, R15, R5: value (none) -> 100
- X2: value (none) -> 32.768KHz
Connections:
- net +3V3: no longer C10.1, C4.1, C5.1, C9.1
- net GND: no longer C10.2, C4.2, C5.2, C9.2

Commit message: updated to USBC connector
Parts:
- removed C3: 20pF, clock:CAP0805
- removed JP3: (no value), pinhead:PINHD-2X2
- removed JP5: (no value), pinhead:PINHD-1X4
- removed R13: 4K7, clock:RESISTOR0805-RES
- removed R14, R15, R5: 100, clock:RESISTOR0805-RES
- removed S1, S2: TAC_SWITCHSMD, SparkFun-Retired:TAC_SWITCHSMD
- removed U$8: TEMT6000, ProtoSnap-v14a:TEMT6000
- removed X3: USB-MICROB, basicBoard:USB-MICROB
- added C10, C15, C20, C22, C24, C4, C5: 100nF, clock:CAP0805
- added C16, C21, C23, C9: 10uF, clock:CAP0805
- added JP6: (no value), pinhead:PINHD-1X5
- added R10, R6: 5.1K, joyAnalog:RESISTOR0805-RES
- added SW1, SW4: 324_SW324_SWITCH_FOOT_HOLE, 3pos_slide_switch:324_SW324_SWITCH_FOOT_HOLE
- added TP5, TP6: TEST-POINT3X5, SparkFun-Passives:TEST-POINT3X5
- added U2: USBC_16P, my_usbc_16p:USBC_16P
- C13, C2: value 47uF -> 10uF; device clock:C-USC1210 -> clock:CAP0805
Connections:
- removed net LIGHT_SENSOR_OUTPUT: IC1PORTA_L.PA1, R13.2, U$8.E1
- removed net N$17: IC1PORTB_L.PB3, R5.1
- removed net N$19: IC1PORTB_L.PB5, R15.1
- removed net N$20: IC1PORTB_L.PB4, R14.1
- removed net PB10: IC1PORTB_H.PB10, JP5.1
- removed net PB11: IC1PORTB_H.PB11, JP5.2
- new net N$16: IC1PORTB_H.PB10, JP6.3
- new net N$22: IC1PORTB_H.PB11, TP5.1
- new net N$23: IC1PORTA_L.PA1, TP6.1
- new net N$31: R6.1, U2.CC2
- new net N$33: R10.1, U2.CC1
- net +3V3: now also C10.1, C14.1, C15.1, C16.1, C20.1, C21.1, C22.1, C23.1, C24.1, C5.1, C9.1, JP6.2, SW1.1, SW1.4; no longer C3.1, JP3.3, JP5.4, S1.3, S1.4, U$8.C1
- net +5V: now also C4.1, U2.VBUS; no longer C14.1, X3.VBUS
- net GND: now also C10.2, C15.2, C16.2, C20.2, C21.2, C22.2, C23.2, C24.2, C4.2, C5.2, C9.2, JP6.1, R10.2, R6.2, SW4.1, SW4.4, U2.GND; no longer C3.2, JP3.1, JP5.3, R13.1, S2.3, S2.4, X3.GND
- net N$3: now also SW4.2, SW4.3; no longer S2.1, S2.2
- net N$5: now also SW1.2, SW1.3; no longer S1.1, S1.2
- net SPI1_MISO: now also IC1PORTB_L.PB4; no longer R14.2
- net SPI1_MOSI: now also IC1PORTB_L.PB5; no longer R15.2
- net SPI1_SCK: now also IC1PORTB_L.PB3; no longer R5.2
- net SWCLK: now also JP6.5; no longer JP3.4
- net SWDIO: now also JP6.4; no longer JP3.2
- net USB_DM: now also U2.DN1, U2.DN2; no longer X3.D-
- net USB_DP: now also U2.DP1, U2.DP2; no longer X3.D+
Other:
- moved on the sheet: C14

Commit message: fixed a silkscreen error on PCB
Parts:
- C18, C19: value (none) -> 47nF
- R11, R12: value 10 -> 1K
Changed lines of the file:
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@@
 <part name="U$15" library="touch_pad" deviceset="TOUCHPAD" device=""/>
 <part name="GND42" library="backplane" deviceset="GND" device=""/>
-<part name="C18" library="clock" deviceset="CAP" device="0805"/>
+<part name="C18" library="clock" deviceset="CAP" device="0805" value="47nF"/>
 <part name="GND43" library="backplane" deviceset="GND" device=""/>
-<part name="R11" library="clock" deviceset="RESISTOR" device="0805-RES" value="10"/>
-<part name="R12" library="clock" deviceset="RESISTOR" device="0805-RES" value="10"/>
-<part name="C19" library="clock" deviceset="CAP" device="0805"/>
+<part name="R11" library="clock" deviceset="RESISTOR" device="0805-RES" value="1K"/>
+<part name="R12" library="clock" deviceset="RESISTOR" device="0805-RES" value="1K"/>
+<part name="C19" library="clock" deviceset="CAP" device="0805" value="47nF"/>
 <part name="GND44" library="backplane" deviceset="GND" device=""/>
 <part name="L1" library="basicBoard" deviceset="INDUCTOR" device="0805" value="33nH"/>
